File: hardware/hardware.kicad_pcb (KiCad board)
At the start: 2 copper layers, 25 parts, among them CON1 BARREL_JACK, J1 MicroSD, P1 FTDI ESP, P2 PPD42NS, P3 DHT22, P4 Fan, P5 I2C, P6 CONN_01X02, Q1 IRF7401, SW1 Reset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

Commit message: pcb of the first production run
Parts:
- added C3: 100n, Capacitors_SMD:C_0805_HandSoldering, F.Cu at (166.1, 117.5)
- added C4: 100n, Capacitors_SMD:C_0805_HandSoldering, B.Cu at (171.2, 117.5)
- added REF**: MountingHole_3mm, Mounting_Holes:MountingHole_3mm, F.Cu at (169.7, 137.8)
- added REF**: MountingHole_3mm, Mounting_Holes:MountingHole_3mm, F.Cu at (190.5, 116.5)
- added REF**: Symbol_OSHW-Logo_SilkScreen, Symbols:Symbol_OSHW-Logo_SilkScreen, B.Cu at (185.7, 137.3)
- CON1: value BARREL_JACK -> Power
- P6: value CONN_01X02 -> 5-9V
- moved F1 6.60 mm to (175.8, 141.4), turned to 180 degrees
- moved Q1 1.52 mm to (185.4, 125.6)
- moved R5 1.14 mm to (185.4, 120.5)
Routing:
- net Net-(Q1-Pad4): track 0.00 -> 11.3 mm
- net +9V: track 41.3 -> 48.0 mm
- net VCC: track 109.2 -> 115.0 mm
- net Net-(D1-Pad2): track 15.1 -> 9.36 mm
- net Net-(P3-Pad2): track 24.3 -> 27.7 mm
- net GND: track 24.9 -> 28.2 mm, vias 5 -> 6
- net Net-(C1-Pad1): track 17.7 -> 16.0 mm
Other:
- board outline added: 44.2 x 44.2 mm
- board text added: "PM Sensor Rev 1 CC BY-SA 4.0 https://github.com/ tiefpunkt/airqualitystation"
